Commit message: Imported upstream version '0.0.4' of 'upstream'

File: kingfisher_description/urdf/standard.urdf.xacro (robot description, xacro)
@@ -10,7 +10,7 @@
     <gazebo>
         <plugin name="kingfisher_imu" filename="libgazebo_ros_imu.so">
-            <updateRate>100.0</updateRate>
+            <updateRate>20.0</updateRate>
             <bodyName>base_link</bodyName>
-            <topicName>raw_imu</topicName>
+            <topicName>imu/data</topicName>
             <rpyOffsets>0 0 0</rpyOffsets> <!-- deprecated -->
             <gaussianNoise>0</gaussianNoise> <!-- deprecated -->
@@ -21,4 +21,18 @@
             <headingDrift>0.1</headingDrift>
             <headingGaussianNoise>0.05</headingGaussianNoise>
+        </plugin>
+    </gazebo>
+    <!-- Set up gps configuration -->
+    <gazebo>
+        <plugin name="kingfisher_gps" filename="libkingfisher_ros_gps.so">
+            <alwaysOn>true</alwaysOn>
+            <updateRate>10.0</updateRate>
+            <bodyName>base_link</bodyName>
+            <topicName>navsat/fix</topicName>
+            <velocityTopicName>navsat/vel</velocityTopicName>
+            <drift>5.0 5.0 5.0</drift>
+            <gaussianNoise>0.1 0.1 0.1</gaussianNoise>
+            <velocityDrift>0 0 0</velocityDrift>
+            <velocityGaussianNoise>0.1 0.1 0.1</velocityGaussianNoise>
         </plugin>
     </gazebo>
@@ -75,3 +89,57 @@
         </sensor>
     </gazebo>
+    <xacro:if value="$(arg sonar_enabled)">
+        <!-- Set up sonar linkage and configuration -->
+        <joint name="base_link_sonar_link_joint" type="fixed">
+        <origin xyz="0 0 -0.2" rpy="0 1.57 0" />
+            <parent link="base_link"/>
+            <child link="sonar_link" />
+        </joint>
+        <link name="sonar_link">
+            <inertial>
+                <mass value="1"/>
+                <origin xyz="0 0 0"/>
+                <inertia ixx="0.1" ixy="0.0" ixz="0.0" iyy="0.1" iyz="0.0" izz="0.1"/>
+            </inertial>
+        </link>
+        <gazebo reference="sonar_link">
+            <sensor type="ray" name="sonar_sensor">
+                <pose>0 0 0 0 0 0</pose>
+                <visualize>false</visualize>
+                <update_rate>20</update_rate>
+                <ray>
+                    <scan>
+                        <horizontal>
+                            <samples>3</samples>
+                            <resolution>1</resolution>
+                            <min_angle>${-5*M_PI/180}</min_angle>
+                            <max_angle>${5*M_PI/180}</max_angle>
+                        </horizontal>
+                    </scan>
+                    <range>
+                        <min>0.10</min>
+                        <max>30.0</max>
+                        <resolution>0.01</resolution>
+                    </range>
+                    <noise>
+                        <type>gaussian</type>
+                        <!-- Noise parameters based on published spec for Hokuyo laser
+                             achieving "+-30mm" accuracy at range < 10m.  A mean of 0.0m and
+                             stddev of 0.01m will put 99.7% of samples within 0.03m of the true
+                             reading. -->
+                        <mean>0.0</mean>
+                        <stddev>0.01</stddev>
+                    </noise>
+                </ray>
+                <plugin name="kingfisher_ros_sonar_controller" filename="libkingfisher_ros_sonar.so">
+                    <gaussianNoise>0.005</gaussianNoise>
+                    <topicName>sonar</topicName>
+                    <frameId>sonar_link</frameId>
+                    <offset>0</offset>
+                    <drift>0</drift>
+                    <driftFrequency>0</driftFrequency>
+                </plugin>
+            </sensor>
+        </gazebo>
+    </xacro:if>
 </robot>
